File: PCB/MaquinaSafetyLevel.kicad_pcb (KiCad board)
At the start: 2 copper layers, 100 x 100 mm, 38 parts, among them J1 ICSP, J10 I2C, J2 Control, J3 LEDs, J4 PD4, J5 PD5, J6 PC1, J7 PC2, J8 PC3, J9 AC_Input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

Commit message: V1.1 PCB, as ordered.
Parts:
- removed G***: LOGO, Logo:name
- added G1: LOGO, Logo:name, F.Cu at (100.0, 103.5)
- moved G2 2.55 mm to (95.8, 96.8)
- moved U3 1.00 mm to (91.5, 127.2)
- renumbered G*** to G2
Routing:
- net GND: track 0.00 -> 379.8 mm
- net VCC: track 0.00 -> 248.9 mm
- net RESET: track 0.00 -> 80.3 mm
- net SDA: track 0.00 -> 64.1 mm
- net SCL: track 0.00 -> 62.2 mm
- net PC2: track 0.00 -> 57.7 mm
- net PD5: track 0.00 -> 57.2 mm
- net Net-(C3-Pad1): track 0.00 -> 55.3 mm
- net PC3: track 0.00 -> 53.9 mm
- net Net-(R6-Pad1): track 0.00 -> 51.8 mm
- net BZR: track 0.00 -> 49.4 mm
- net PD4: track 0.00 -> 41.5 mm
- net PC1: track 0.00 -> 37.1 mm
- net Net-(C6-Pad1): track 0.00 -> 34.6 mm
- net Net-(R7-Pad1): track 0.00 -> 33.1 mm
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- added copper zone on B.Cu, net GND
- added copper zone on F.Cu, net GND
Other:
- board text added: "https://github.com/andystopford/SCRAM/tree/master"
